File: pcb/RscDroneBadge.sch (EAGLE design)
At the start: 31 parts, among them Q1 BC547, Q2 BC547, Q3 BC547, Q4 BC547

Commit message: update schematic and board, add drawing
Parts:
- added BAT: CR2032_PLASTIC, BASTL_BATHOLDER:CR2032_PLASTIC
Connections:
- net GND: now also BAT.NEG
- net VDD: now also BAT.POS
Other:
- note added: "Recommended Yellow Leds: L-53SYDK L-53SYD"

Commit message: routing
Parts:
- added ISP: 2X3POGONO_VIA, BASTL_CONNECTORS:2X3POGONO_VIA
Connections:
- removed net N$5: IC1.PB0(MOSI), R1.1
- removed net N$6: IC1.PB1(MISO), R2.1
- removed net N$7: IC1.PB2(SCK/ADC1), R3.1
- new net MISO: IC1.PB1(MISO), ISP.1, R2.1
- new net MOSI: IC1.PB0(MOSI), ISP.4, R1.1
- new net RST: IC1.PB5(NRES), ISP.5
- new net SCK: IC1.PB2(SCK/ADC1), ISP.3, R3.1
- net GND: now also ISP.6
- net VDD: now also ISP.2
Changed lines of the file:
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@@
 <layer number="59" name="tCarbon" color="7" fill="1" visible="no" active="no"/>
 <layer number="60" name="bCarbon" color="7" fill="1" visible="no" active="no"/>
+<layer number="61" name="stand" color="7" fill="1" visible="no" active="no"/>
 <layer number="88" name="SimResults" color="9" fill="1" visible="yes" active="yes"/>
 <layer number="89" name="SimProbes" color="9" fill="1" visible="yes" active="yes"/>
@@
 <layer number="115" name="card" color="7" fill="1" visible="yes" active="yes"/>
 <layer number="116" name="Patch_BOT" color="7" fill="1" visible="yes" active="yes"/>
+<layer number="117" name="mPads" color="7" fill="1" visible="yes" active="yes"/>
 <layer number="118" name="Rect_Pads" color="7" fill="1" visible="yes" active="yes"/>
+<layer number="119" name="mUnrouted" color="7" fill="1" visible="yes" active="yes"/>
 <layer number="120" name="_Dimension" color="7" fill="1" visible="yes" active="yes"/>
 <layer number="121" name="_tsilk" color="7" fill="1" visible="yes" active="yes"/>
@@
 <layer number="131" name="tAdjust" color="7" fill="1" visible="yes" active="yes"/>
 <layer number="132" name="bAdjust" color="7" fill="1" visible="yes" active="yes"/>
+<layer number="133" name="mtFinish" color="7" fill="1" visible="yes" active="yes"/>
+<layer number="134" name="mbFinish" color="7" fill="1" visible="yes" active="yes"/>
 <layer number="135" name="_tanames" color="7" fill="1" visible="yes" active="yes"/>
 <layer number="136" name="_banames" color="7" fill="1" visible="yes" active="yes"/>
 <layer number="137" name="_taDocu" color="7" fill="1" visible="yes" active="yes"/>
 <layer number="138" name="_baDocu" color="7" fill="1" visible="yes" active="yes"/>
+<layer number="139" name="mtKeepout" color="7" fill="1" visible="yes" active="yes"/>
+<layer number="140" name="mbKeepout" color="7" fill="1" visible="yes" active="yes"/>
+<layer number="141" name="mtRestrict" color="7" fill="1" visible="yes" active="yes"/>
+<layer number="142" name="mbRestrict" color="7" fill="1" visible="yes" active="yes"/>
+<layer number="143" name="mvRestrict" color="7" fill="1" visible="yes" active="yes"/>
 <layer number="144" name="Drill_legend" color="7" fill="1" visible="yes" active="yes"/>
 <layer number="145" name="DrillLegend_01-16" color="7" fill="1" visible="yes" active="yes"/>
 <layer number="146" name="DrillLegend_01-20" color="7" fill="1" visible="yes" active="yes"/>
+<layer number="147" name="DrillLegend_01-16" color="7" fill="1" visible="yes" active="yes"/>
+<layer number="148" name="DrillLegend_01-20" color="7" fill="1" visible="yes" active="yes"/>
+<layer number="149" name="DrillLegend_02-15" color="7" fill="1" visible="yes" active="yes"/>
 <layer number="150" name="Notes" color="7" fill="1" visible="yes" active="yes"/>
 <layer number="151" name="HeatSink" color="7" fill="1" visible="yes" active="yes"/>
@@
 <layer number="154" name="FabDoc2" color="7" fill="1" visible="yes" active="yes"/>
 <layer number="155" name="FabDoc3" color="7" fill="1" visible="yes" active="yes"/>
+<layer number="156" name="DXF0409-TOP" color="7" fill="1" visible="yes" active="yes"/>
+<layer number="157" name="DXF0409-BOTTOM" color="7" fill="1" visible="yes" active="yes"/>
 <layer number="160" name="O_Dim" color="7" fill="1" visible="yes" active="yes"/>
+<layer number="166" name="AntennaArea" color="7" fill="1" visible="yes" active="yes"/>
+<layer number="168" name="4mmHeightArea" color="7" fill="1" visible="yes" active="yes"/>
+<layer number="190" name="Faceplate-Hole" color="7" fill="1" visible="yes" active="yes"/>
+<layer number="191" name="mNets" color="7" fill="1" visible="yes" active="yes"/>
+<layer number="192" name="mBusses" color="7" fill="1" visible="yes" active="yes"/>
+<layer number="193" name="mPins" color="7" fill="1" visible="yes" active="yes"/>
+<layer number="194" name="mSymbols" color="7" fill="1" visible="yes" active="yes"/>
+<layer number="195" name="mNames" color="7" fill="1" visible="yes" active="yes"/>
+<layer number="196" name="mValues" color="7" fill="1" visible="yes" active="yes"/>
 <layer number="199" name="Contour" color="7" fill="1" visible="yes" active="yes"/>
 <layer number="200" name="200bmp" color="7" fill="1" visible="yes" active="yes"/>
@@
 <part name="SUPPLY3" library="BASTL_SYMBOLS" library_urn="urn:adsk.eagle:library:32975873" deviceset="VDD" device=""/>
 <part name="GND7" library="BASTL_SYMBOLS" library_urn="urn:adsk.eagle:library:32975873" deviceset="GND" device=""/>
+<part name="ISP" library="BASTL_CONNECTORS" library_urn="urn:adsk.eagle:library:32904192" deviceset="2X3POGO" device="NO_VIA" package3d_urn="urn:adsk.eagle:package:32904263/1"/>
+<part name="GND8" library="BASTL_SYMBOLS" library_urn="urn:adsk.eagle:library:32975873" deviceset="GND" device=""/>
+<part name="SUPPLY4" library="BASTL_SYMBOLS" library_urn="urn:adsk.eagle:library:32975873" deviceset="VDD" device=""/>
 </parts>
 <sheets>
@@
 <attribute name="VALUE" x="-2.54" y="53.34" size="1.778" layer="96"/>
 </instance>
+<instance part="ISP" gate="G$1" x="38.1" y="96.52" smashed="yes">
+<attribute name="NAME" x="35.56" y="102.362" size="1.778" layer="95"/>
+</instance>
+<instance part="GND8" gate="1" x="45.72" y="91.44" smashed="yes">
+<attribute name="VALUE" x="43.18" y="88.9" size="1.778" layer="96"/>
+</instance>
+<instance part="SUPPLY4" gate="G$1" x="45.72" y="101.6" smashed="yes">
+<attribute name="VALUE" x="43.815" y="104.775" size="1.778" layer="96"/>
+</instance>
 </instances>
 <busses>
@@
 <pinref part="GND7" gate="1" pin="GND"/>
 </segment>
+<segment>
+<pinref part="ISP" gate="G$1" pin="6"/>
+<pinref part="GND8" gate="1" pin="GND"/>
+</segment>
 </net>
 <net name="N$2" class="0">
@@
 <pinref part="Q3" gate="G$1" pin="B"/>
 <pinref part="R3" gate="G$1" pin="2"/>
-</segment>
-</net>
-<net name="N$5" class="0">
-<segment>
-<pinref part="IC1" gate="G$1" pin="PB0(MOSI)"/>
-<wire x1="50.8" y1="71.12" x2="58.42" y2="71.12" width="0.1524" layer="91"/>
-<wire x1="58.42" y1="71.12" x2="58.42" y2="78.74" width="0.1524" layer="91"/>
-<pinref part="R1" gate="G$1" pin="1"/>
-</segment>
-</net>
-<net name="N$6" class="0">
-<segment>
-<pinref part="IC1" gate="G$1" pin="PB1(MISO)"/>
-<pinref part="R2" gate="G$1" pin="1"/>
-<wire x1="50.8" y1="68.58" x2="93.98" y2="68.58" width="0.1524" layer="91"/>
-<wire x1="93.98" y1="68.58" x2="93.98" y2="78.74" width="0.1524" layer="91"/>
-</segment>
-</net>
-<net name="N$7" class="0">
-<segment>
-<pinref part="IC1" gate="G$1" pin="PB2(SCK/ADC1)"/>
-<pinref part="R3" gate="G$1" pin="1"/>
-<wire x1="50.8" y1="66.04" x2="129.54" y2="66.04" width="0.1524" layer="91"/>
-<wire x1="129.54" y1="66.04" x2="129.54" y2="78.74" width="0.1524" layer="91"/>
 </segment>
 </net>
@@
 <pinref part="SUPPLY3" gate="G$1" pin="VDD"/>
 </segment>
+<segment>
+<pinref part="ISP" gate="G$1" pin="2"/>
+<pinref part="SUPPLY4" gate="G$1" pin="VDD"/>
+</segment>
 </net>
 <net name="N$14" class="0">
@@
 </segment>
 </net>
+<net name="MISO" class="0">
+<segment>
+<pinref part="ISP" gate="G$1" pin="1"/>
+<wire x1="30.48" y1="99.06" x2="27.94" y2="99.06" width="0.1524" layer="91"/>
+<label x="27.94" y="99.06" size="1.27" layer="95" rot="R180" xref="yes"/>
+</segment>
+<segment>
+<pinref part="IC1" gate="G$1" pin="PB1(MISO)"/>
+<pinref part="R2" gate="G$1" pin="1"/>
+<wire x1="50.8" y1="68.58" x2="93.98" y2="68.58" width="0.1524" layer="91"/>
+<wire x1="93.98" y1="68.58" x2="93.98" y2="78.74" width="0.1524" layer="91"/>
+<label x="68.58" y="68.58" size="1.27" layer="95" rot="R90" xref="yes"/>
+</segment>
+</net>
+<net name="SCK" class="0">
+<segment>
+<pinref part="ISP" gate="G$1" pin="3"/>
+<wire x1="30.48" y1="96.52" x2="27.94" y2="96.52" width="0.1524" layer="91"/>
+<label x="27.94" y="96.52" size="1.27" layer="95" rot="R180" xref="yes"/>
+</segment>
+<segment>
+<pinref part="IC1" gate="G$1" pin="PB2(SCK/ADC1)"/>
+<pinref part="R3" gate="G$1" pin="1"/>
+<wire x1="50.8" y1="66.04" x2="129.54" y2="66.04" width="0.1524" layer="91"/>
+<wire x1="129.54" y1="66.04" x2="129.54" y2="78.74" width="0.1524" layer="91"/>
+<label x="99.06" y="66.04" size="1.27" layer="95" rot="R90" xref="yes"/>
+</segment>
+</net>
+<net name="RST" class="0">
+<segment>
+<pinref part="ISP" gate="G$1" pin="5"/>
+<wire x1="30.48" y1="93.98" x2="27.94" y2="93.98" width="0.1524" layer="91"/>
+<label x="27.94" y="93.98" size="1.27" layer="95" rot="R180" xref="yes"/>
+</segment>
+<segment>
+<wire x1="50.8" y1="58.42" x2="50.8" y2="55.88" width="0.1524" layer="91"/>
+<pinref part="IC1" gate="G$1" pin="PB5(NRES)"/>
+<label x="50.8" y="55.88" size="1.27" layer="95" xref="yes"/>
+</segment>
+</net>
+<net name="MOSI" class="0">
+<segment>
+<pinref part="ISP" gate="G$1" pin="4"/>
+<wire x1="45.72" y1="96.52" x2="48.26" y2="96.52" width="0.1524" layer="91"/>
+<label x="48.26" y="96.52" size="1.27" layer="95" xref="yes"/>
+</segment>
+<segment>
+<pinref part="IC1" gate="G$1" pin="PB0(MOSI)"/>
+<wire x1="50.8" y1="71.12" x2="58.42" y2="71.12" width="0.1524" layer="91"/>
+<wire x1="58.42" y1="71.12" x2="58.42" y2="78.74" width="0.1524" layer="91"/>
+<pinref part="R1" gate="G$1" pin="1"/>
+<label x="58.42" y="71.12" size="1.27" layer="95" xref="yes"/>
+</segment>
+</net>

Commit message: finishing
Parts:
- BAT: value CR2032_PLASTIC -> CR2032 HOLDER
- IC1: value (none) -> ATTINY85
- S1: value PUSH_MOMENTARY_THT_6X6MM -> 6x6mm BUTTON
Changed lines of the file:
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@@
 </classes>
 <parts>
-<part name="IC1" library="BASTL_ICS" library_urn="urn:adsk.eagle:library:32977748" deviceset="ATTINY85" device="-20PU" package3d_urn="urn:adsk.eagle:package:43822317/1"/>
-<part name="S1" library="BASTL_SWITCHES" library_urn="urn:adsk.eagle:library:32903743" deviceset="PUSH_MOMENTARY" device="_THT_6X6MM" package3d_urn="urn:adsk.eagle:package:32903802/2"/>
+<part name="IC1" library="BASTL_ICS" library_urn="urn:adsk.eagle:library:32977748" deviceset="ATTINY85" device="-20PU" package3d_urn="urn:adsk.eagle:package:43822317/1" value="ATTINY85"/>
+<part name="S1" library="BASTL_SWITCHES" library_urn="urn:adsk.eagle:library:32903743" deviceset="PUSH_MOMENTARY" device="_THT_6X6MM" package3d_urn="urn:adsk.eagle:package:32903802/2" value="6x6mm BUTTON"/>
 <part name="GND1" library="BASTL_SYMBOLS" library_urn="urn:adsk.eagle:library:32975873" deviceset="GND" device=""/>
 <part name="Q1" library="BASTL_TRANZISTORS" library_urn="urn:adsk.eagle:library:32975847" deviceset="BC547" device="" package3d_urn="urn:adsk.eagle:package:43822007/4"/>
@@
 <part name="SUPPLY2" library="BASTL_SYMBOLS" library_urn="urn:adsk.eagle:library:32975873" deviceset="VDD" device=""/>
 <part name="C1" library="BASTL_CAPACITORS" library_urn="urn:adsk.eagle:library:32978038" deviceset="CAPACITOR_THT" device="_2.54" package3d_urn="urn:adsk.eagle:package:43822030/2" value="100n"/>
-<part name="BAT" library="BASTL_BATHOLDER" library_urn="urn:adsk.eagle:library:32978091" deviceset="CR2032_PLASTIC" device="" package3d_urn="urn:adsk.eagle:package:43822280/2"/>
+<part name="BAT" library="BASTL_BATHOLDER" library_urn="urn:adsk.eagle:library:32978091" deviceset="CR2032_PLASTIC" device="" package3d_urn="urn:adsk.eagle:package:43822280/2" value="CR2032 HOLDER"/>
 <part name="SUPPLY3" library="BASTL_SYMBOLS" library_urn="urn:adsk.eagle:library:32975873" deviceset="VDD" device=""/>
 <part name="GND7" library="BASTL_SYMBOLS" library_urn="urn:adsk.eagle:library:32975873" deviceset="GND" device=""/>

Commit message: remove "85" from ATTINY label on the board
Parts:
- IC1: value ATTINY85 -> ATTINY
Changed lines of the file:
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@@
 </classes>
 <parts>
-<part name="IC1" library="BASTL_ICS" library_urn="urn:adsk.eagle:library:32977748" deviceset="ATTINY85" device="-20PU" package3d_urn="urn:adsk.eagle:package:43822317/1" value="ATTINY85"/>
+<part name="IC1" library="BASTL_ICS" library_urn="urn:adsk.eagle:library:32977748" deviceset="ATTINY85" device="-20PU" package3d_urn="urn:adsk.eagle:package:43822317/1" value="ATTINY"/>
 <part name="S1" library="BASTL_SWITCHES" library_urn="urn:adsk.eagle:library:32903743" deviceset="PUSH_MOMENTARY" device="_THT_6X6MM" package3d_urn="urn:adsk.eagle:package:32903802/2" value="6x6mm BUTTON"/>
 <part name="GND1" library="BASTL_SYMBOLS" library_urn="urn:adsk.eagle:library:32975873" deviceset="GND" device=""/>
